File: PCB2024/Baja Dashboard Schematic Part 2 abc/Baja Dashboard Schematic Part 2.kicad_pcb (KiCad board)
At the start: 4 copper layers, 145.5 x 72 mm, 53 parts, among them J1 Conn_01x04_Pin, J2 Conn_01x02_Pin, Q2 MMBT2222_, SW1 SW_Push, SW2 SW_Push, U1 TLC5917, U2 TLC5917, U3 TLC5917, U9 TLC555xPS

Commit message: Add files via upload
Parts:
- J2: value Conn_01x02_Pin -> Conn_01x04_Pin; footprint Connector_PinHeader_1.00mm:PinHeader_1x02_P1.00mm_Vertical -> bajaRedoSaves:PowerBoard
- moved J2 27.4 mm to (150.5, 82.8), turned to 90 degrees
Routing:
- net +12V: track 0.00 -> 43.6 mm, vias 0 -> 1
- net +5V: track 62.4 -> 54.8 mm, vias 7 -> 6
- net /D12LED: track 53.0 -> 56.6 mm, vias 1 -> 0
- net /DCU8Left: track 112.7 -> 113.9 mm
- net /D13LED: track 50.8 -> 51.5 mm
