File: PCB2024/Baja Dashboard Schematic Part 2 abc/Baja Dashboard Schematic Part 2.kicad_sch (KiCad schematic)
At the start: 53 parts, among them J1 Conn_01x04_Pin, J2 Conn_01x02_Pin, Q2 MMBT2222_, SW1 SW_Push, SW2 SW_Push, U1 TLC5917, U2 TLC5917, U3 TLC5917, U9 TLC555xPS

Commit message: Add files via upload
Parts:
- removed J2: Conn_01x02_Pin, Connector_PinHeader_1.00mm:PinHeader_1x02_P1.00mm_Vertical, symbol Connector:Conn_01x02_Pin
- added J2: Conn_01x04_Pin, bajaRedoSaves:PowerBoard, symbol Connector:Conn_01x04_Pin
Connections:
- net +12V: now also J2.3 (Pin_3)
- net +5V: now also J2.1 (Pin_1)
- net GND: now also J2.2 (Pin_2), J2.4 (Pin_4)
