File: PCB/Baja Dashboard Schematic Part 2 abc/Baja Dashboard Schematic Part 2.kicad_pcb (KiCad board)
At the start: 4 copper layers, 145.5 x 72 mm, 53 parts, among them J1 Conn_01x04_Pin, J2 Conn_01x04_Pin, Q2 MMBT2222_, SW1 SW_Push, SW2 SW_Push, U1 TLC5917, U2 TLC5917, U3 TLC5917, U9 TLC555xPS

Commit message: Add files via upload
Parts:
- removed Q2: MMBT2222_, bajaRedoSaves:MMBT2222
- added Q1: MMBT2222_, bajaRedoSaves:MMBT2222, B.Cu at (202.4, 94.0)
- C1: value C -> 10nF
- C2: value C -> 10^pF
- R1: value R -> 200
- R2, R3: value R -> 300
- moved C1 5.94 mm to (183.8, 89.5), turned to 180 degrees
- moved C2 1.54 mm to (195.2, 87.0), turned to 0 degrees
- moved R2 0.80 mm to (184.8, 86.3)
- moved R3 0.77 mm to (194.3, 88.5)
- moved R1 0.75 mm to (184.5, 87.8)
Connections:
- C1 pad 2: Net-(Q1-C) -> GND
- C2 pad 2: Net-(Q1-C) -> GND
- R2 pad 1: +5V -> Net-(U9-R)
- U9 pad 1: Net-(U9-GND) -> GND
- U9 pad 4: +5V -> Net-(U9-R)
- U9 pad 8: +5V -> Net-(U9-R)
Routing:
- net Net-(U9-R): track 0.00 -> 23.8 mm, vias 0 -> 2
- net Net-(U9-THR): track 32.1 -> 10.6 mm
- net Net-(U9-GND): track 17.9 -> 0.00 mm
- net Net-(Q1-C): track 13.3 -> 0.00 mm, vias 2 -> 0
- net +5V: track 54.8 -> 65.6 mm
- net Net-(LS1-Pad1): track 85.2 -> 91.1 mm
- net GND: track 21.4 -> 26.5 mm
- net Net-(U9-CV): track 3.25 -> 2.07 mm
- net Net-(Q1-PadB): track 3.50 -> 2.70 mm
- net Net-(U9-Q): track 1.89 -> 2.64 mm
